File: base/base.kicad_pcb (KiCad board)
At the start: 2 copper layers, 29 x 16 mm, 2 parts, among them J1 Conn_01x08, J2 Conn_02x03

Commit message: everything else
Parts:
- J2: moved to F.Cu
- moved J2 2.53 mm to (183.2, 138.5), turned to 0 degrees
Other:
- board text added: "SIG_IN"
- board text added: "VCC"
