File: blaster/ir_shotgun.kicad_pcb (KiCad board)
At the start: 2 copper layers, 14.2 x 21 mm, 18 parts, among them J1 Conn_02x03, Q1 AO3400A

Commit message: everything else
Parts:
- moved J1 0.07 mm to (115.6, 73.0)
Routing:
- net GND: track 0.00 -> 8.67 mm, vias 0 -> 4
- added copper zone on F.Cu, net GND
Changed lines of the file:
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@@
 	(footprint "Connector_PinHeader_2.54mm:PinHeader_2x03_P2.54mm_Vertical"
 		(layer "B.Cu")
-		(at 115.670001 72.975 -90)
+		(at 115.600001 72.975 -90)
 		(descr "Through hole straight pin header, 2x03, 2.54mm pitch, double rows")
 		(tags "Through hole pin header THT 2x03 2.54mm double row")
@@
 		)
 		(fp_text user "${REFERENCE}"
-			(at 1.27 -2.54 180)
+			(at 1.27 -2.54 0)
 			(layer "B.Fab")
 			(effects
@@
 		(embedded_fonts no)
 		(model "${KICAD9_3DMODEL_DIR}/Connector_PinHeader_2.54mm.3dshapes/PinHeader_2x03_P2.54mm_Vertical.wrl"
+			(hide yes)
 			(offset
 				(xyz 0 0 0)
@@
 			)
 			(rotate
-				(xyz 0 0 0)
+				(xyz -0 -0 -0)
+			)
+		)
+		(model "G:/KiCad/Projects/ir_shotgun/connector.step"
+			(offset
+				(xyz 1.25 0 2.5)
+			)
+			(scale
+				(xyz 1 1 1)
+			)
+			(rotate
+				(xyz 90 -0 -90)
 			)
 		)
@@
 		(net 1)
 	)
-	(segment
-		(start 115.670001 72.975)
-		(end 115.670001 75.515)
-		(width 0.8)
-		(layer "B.Cu")
-		(net 3)
-	)
-	(segment
-		(start 113 65.1625)
-		(end 113 70.304999)
+	(via
+		(at 118 68.25)
+		(size 0.5)
+		(drill 0.3)
+		(layers "F.Cu" "B.Cu")
+		(net 2)
+	)
+	(via
+		(at 114.25 61.75)
+		(size 0.5)
+		(drill 0.3)
+		(layers "F.Cu" "B.Cu")
+		(net 2)
+	)
+	(via
+		(at 118 64)
+		(size 0.5)
+		(drill 0.3)
+		(layers "F.Cu" "B.Cu")
+		(net 2)
+	)
+	(via
+		(at 118 62.25)
+		(size 0.5)
+		(drill 0.3)
+		(layers "F.Cu" "B.Cu")
+		(net 2)
+	)
+	(segment
+		(start 115 63.300001)
+		(end 115 62.5)
+		(width 0.8)
+		(layer "B.Cu")
+		(net 2)
+	)
+	(segment
+		(start 115 63.300001)
+		(end 117.300001 63.300001)
+		(width 0.8)
+		(layer "B.Cu")
+		(net 2)
+	)
+	(segment
+		(start 117.300001 63.300001)
+		(end 118 64)
+		(width 0.8)
+		(layer "B.Cu")
+		(net 2)
+	)
+	(segment
+		(start 117.741161 68.508839)
+		(end 118 68.25)
+		(width 0.8)
+		(layer "B.Cu")
+		(net 2)
+	)
+	(segment
+		(start 116.334664 68.508839)
+		(end 117.741161 68.508839)
+		(width 0.8)
+		(layer "B.Cu")
+		(net 2)
+	)
+	(segment
+		(start 118 60.5)
+		(end 118 62.25)
+		(width 0.8)
+		(layer "B.Cu")
+		(net 2)
+	)
+	(segment
+		(start 115 62.5)
+		(end 114.25 61.75)
+		(width 0.8)
+		(layer "B.Cu")
+		(net 2)
+	)
+	(segment
+		(start 113 70.374999)
+		(end 113 65.1625)
 		(width 0.8)
 		(layer "B.Cu")
@@
 	)
 	(segment
-		(start 113 70.304999)
-		(end 115.670001 72.975)
+		(start 115.600001 75.515)
+		(end 115.600001 72.975)
+		(width 0.8)
+		(layer "B.Cu")
+		(net 3)
+	)
+	(segment
+		(start 115.600001 72.975)
+		(end 113 70.374999)
 		(width 0.8)
 		(layer "B.Cu")
@@
 			)
 		)
+	)
+	(zone
+		(net 2)
+		(net_name "GND")
+		(layer "F.Cu")
+		(hatch edge 0.5)
+		(priority 2)
+		(connect_pads yes
+			(clearance 0.5)
+		)
+		(min_thickness 0.25)
+		(filled_areas_thickness no)
+		(fill yes
+			(thermal_gap 0.5)
+			(thermal_bridge_width 0.5)
+		)
+		(polygon
+			(pts
+				(xy 111.25 59.25) (xy 111.25 69.25) (xy 125 69.25) (xy 125 59.25)
+			)
+		)
